File: convention_badge_kicad/convention_badge_pcb_v2/convention_badge_pcb_v2.kicad_sch (KiCad schematic)
At the start: 48 parts, among them J1 USBC, J2 Conn_01x03_Pin, J3 3.7V Battery, J4 Conn_01x07_Pin, J5 Conn_01x07_Pin, Q1 AO3401A, SW1 SW4X2, SW2 SW4X2, SW3 SW_Push, SW4 SW_Push, SW5 SW_Push, SW6 SW4X2, U1 ESP32-C3-WROOM-02, U2 FS8205A, U3 TP4056, U4 DW01A, U5 TLV75733PDBV

Commit message: add readme content, modify pins in code for C3
Connections:
- net GND: now also R9.1, U2.1 (S1)
Changed lines of the file:
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@@
 	)
 	(junction
+		(at 195.58 57.15)
+		(diameter 0)
+		(color 0 0 0 0)
+	)
+	(junction
 		(at 138.43 72.39)
 		(diameter 0)
@@
 	(wire
 		(pts
+			(xy 195.58 57.15) (xy 195.58 60.96)
+		)
+		(stroke
+			(width 0)
+			(type default)
+		)
+	)
+	(wire
+		(pts
 			(xy 129.54 72.39) (xy 129.54 80.01)
 		)
@@
 					(unit 1)
 				)
+			)
+		)
+	)
+	(symbol
+		(lib_id "power:GND")
+		(at 195.58 60.96 0)
+		(unit 1)
+		(exclude_from_sim no)
+		(in_bom yes)
+		(on_board yes)
+		(dnp no)
+		(property "Reference" "#PWR030"
+			(at 195.58 67.31 0)
+			(effects
+				(font
+					(size 1.27 1.27)
+				)
+				(hide yes)
+			)
+		)
+		(property "Value" "GND"
+			(at 195.58 65.024 0)
+			(effects
+				(font
+					(size 1.27 1.27)
+				)
+			)
+		)
+		(property "Footprint" ""
+			(at 195.58 60.96 0)
+			(effects
+				(font
+					(size 1.27 1.27)
+				)
+				(hide yes)
+			)
+		)
+		(property "Datasheet" ""
+			(at 195.58 60.96 0)
+			(effects
+				(font
+					(size 1.27 1.27)
+				)
+				(hide yes)
+			)
+		)
+		(property "Description" "Power symbol creates a global label with name \"GND\" , ground"
+			(at 195.58 60.96 0)
+			(effects
+				(font
+					(size 1.27 1.27)
+				)
+				(hide yes)
+			)
+		)
+		(pin "1"
+		)
+		(instances
+			(project "convention_badge_pcb_v2"
+				(path "/78d9d3f2-d4fd-4baf-b65f-a1e04a215bde"
+					(reference "#PWR030")
+					(unit 1)
+				)
