File: convention_badge_kicad/convention_badge_pcb_v2/convention_badge_pcb_v2.kicad_sch (KiCad schematic)
At the start: 48 parts, among them J1 USBC, J2 Conn_01x03_Pin, J3 3.7V Battery, J4 Conn_01x07_Pin, J5 Conn_01x07_Pin, Q1 AO3401A, SW1 SW4X2, SW2 SW4X2, SW3 SW_Push, SW4 SW_Push, SW5 SW_Push, SW6 SW4X2, U1 ESP32-C3-WROOM-02, U2 FS8205A, U3 TP4056, U4 DW01A, U5 TLV75733PDBV

Commit message: made reworked changes in schematic and layout
Parts:
- added C12: 100uF, PCM_JLCPCB:C_CASE-B-3528-21(mm), symbol Device:C_Small_US
Connections:
- net +3.3V: now also C12.1
- net GND: now also C12.2
- net VBAT: now also Q1.3 (D); no longer Q1.1 (D)
- net VUSB: now also Q1.1 (G); no longer Q1.2 (G)
- net at C6.1, D3.1 (K), U5.1 (IN)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: now also Q1.2 (S); no longer Q1.3 (S)
Changed lines of the file:
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@@
 	)
 	(junction
+		(at 59.69 92.71)
+		(diameter 0)
+		(color 0 0 0 0)
+	)
+	(junction
 		(at 129.54 72.39)
 		(diameter 0)
@@
 	)
 	(junction
+		(at 77.47 93.98)
+		(diameter 0)
+		(color 0 0 0 0)
+	)
+	(junction
 		(at 34.29 179.07)
 		(diameter 0)
@@
 	(wire
 		(pts
+			(xy 74.93 102.87) (xy 74.93 93.98)
+		)
+		(stroke
+			(width 0)
+			(type default)
+		)
+	)
+	(wire
+		(pts
 			(xy 110.49 35.56) (xy 118.11 35.56)
 		)
@@
 	(wire
 		(pts
+			(xy 72.39 102.87) (xy 74.93 102.87)
+		)
+		(stroke
+			(width 0)
+			(type default)
+		)
+	)
+	(wire
+		(pts
 			(xy 15.24 29.21) (xy 21.59 29.21)
 		)
@@
 	(wire
 		(pts
+			(xy 63.5 102.87) (xy 63.5 96.52)
+		)
+		(stroke
+			(width 0)
+			(type default)
+		)
+	)
+	(wire
+		(pts
 			(xy 168.91 58.42) (xy 171.45 58.42)
 		)
@@
 	(wire
 		(pts
+			(xy 59.69 96.52) (xy 59.69 92.71)
+		)
+		(stroke
+			(width 0)
+			(type default)
+		)
+	)
+	(wire
+		(pts
 			(xy 123.19 72.39) (xy 129.54 72.39)
 		)
@@
 	(wire
 		(pts
+			(xy 74.93 93.98) (xy 77.47 93.98)
+		)
+		(stroke
+			(width 0)
+			(type default)
+		)
+	)
+	(wire
+		(pts
 			(xy 52.07 116.84) (xy 60.96 116.84)
 		)
@@
 	(wire
 		(pts
+			(xy 63.5 96.52) (xy 59.69 96.52)
+		)
+		(stroke
+			(width 0)
+			(type default)
+		)
+	)
+	(wire
+		(pts
 			(xy 77.47 54.61) (xy 86.36 54.61)
 		)
@@
 	(wire
 		(pts
+			(xy 67.31 102.87) (xy 63.5 102.87)
+		)
+		(stroke
+			(width 0)
+			(type default)
+		)
+	)
+	(wire
+		(pts
 			(xy 15.24 36.83) (xy 21.59 36.83)
 		)
@@
 	)
 	(symbol
+		(lib_id "Device:C_Small_US")
+		(at 69.85 102.87 90)
+		(unit 1)
+		(exclude_from_sim no)
+		(in_bom yes)
+		(on_board yes)
+		(dnp no)
+		(fields_autoplaced yes)
+		(property "Reference" "C12"
+			(at 69.977 96.52 90)
+			(effects
+				(font
+					(size 1.27 1.27)
+				)
+			)
+		)
+		(property "Value" "100uF"
+			(at 69.977 99.06 90)
+			(effects
+				(font
+					(size 1.27 1.27)
+				)
+			)
+		)
+		(property "Footprint" "PCM_JLCPCB:C_CASE-B-3528-21(mm)"
+			(at 69.85 102.87 0)
+			(effects
+				(font
+					(size 1.27 1.27)
+				)
+				(hide yes)
+			)
+		)
+		(property "Datasheet" ""
+			(at 69.85 102.87 0)
+			(effects
+				(font
+					(size 1.27 1.27)
+				)
+				(hide yes)
+			)
+		)
+		(property "Description" "capacitor, small US symbol"
+			(at 69.85 102.87 0)
+			(effects
+				(font
+					(size 1.27 1.27)
+				)
+				(hide yes)
+			)
+		)
+		(property "LCSC" "C122271"
+			(at 69.85 102.87 0)
+			(effects
+				(font
+					(size 1.27 1.27)
+				)
+				(hide yes)
+			)
+		)
+		(pin "1"
+		)
+		(pin "2"
+		)
+		(instances
+			(project "convention_badge_pcb_v2"
+				(path "/78d9d3f2-d4fd-4baf-b65f-a1e04a215bde"
+					(reference "C12")
+					(unit 1)
+				)
+			)
+		)
+	)
+	(symbol
 		(lib_id "Connector:Conn_01x07_Pin")
 		(at 123.19 30.48 180)
@@
 			)
 		)
-		(property "Sim.Pins" "1=D 2=G 3=S"
+		(property "Sim.Pins" "1=G 2=S 3=D"
 			(at 133.35 74.93 0)
 			(effects
