File: convention_badge_kicad/convention_badge_pcb_v2/convention_badge_pcb_v2.kicad_pcb (KiCad board)
At the start: 4 copper layers, 90 x 98 mm, 56 parts, among them J1 USBC, J2 Conn_01x03_Pin, J3 3.7V Battery, J4 Conn_01x07_Pin, J5 Conn_01x07_Pin, Q1 AO3401A, SW1 SW4X2, SW2 SW4X2, SW3 SW_Push, SW4 SW_Push, SW5 SW_Push, SW6 SW4X2, U1 ESP32-C3-WROOM-02, U2 FS8205A, U3 TP4056, U4 DW01A, U5 TLV75733PDBV

Commit message: made reworked changes in schematic and layout
Parts:
- added C12: 100uF, PCM_JLCPCB:C_CASE-B-3528-21(mm), B.Cu at (112.0, 108.8)
- moved Q1 0.35 mm to (127.8, 104.2), turned to 90 degrees
Connections:
- Q1 pad 1: /VBAT -> /VUSB
- Q1 pad 2: /VUSB -> Net-(D3-K)
- Q1 pad 3: Net-(D3-K) -> /VBAT
Routing:
- net +3.3V: track 11.4 -> 14.8 mm
- net GND: track 74.3 -> 76.6 mm, vias 26 -> 28
- net Net-(D3-K): track 12.7 -> 14.9 mm
